File: Mini_Tastatur.kicad_pcb (KiCad board)
At the start: 2 copper layers, 56 x 83 mm, 16 parts, among them IC1 74HCT1G125GW,125, SW1 RotaryEncoder_Switch, SW2 SW_Reset, U1 DM-OLED096-636, U10 MX1A-11NN_RGB, U2 MX1A-11NN_RGB, U3 MX1A-11NN_RGB, U4 MX1A-11NN_RGB, U5 MX1A-11NN_RGB, U6 MX1A-11NN_RGB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

Commit message: v2
Parts:
- D10: footprint Diode_SMD:D_MiniMELF -> Diode_SMD:D_SOD-523
- moved U4 52.3 mm to (119.0, 116.0)
- moved U9 41.6 mm to (81.0, 154.0)
- moved U8 41.1 mm to (100.0, 154.0)
- moved U3 26.2 mm to (100.0, 116.0)
- moved U5 26.2 mm to (81.0, 135.0)
- moved U7 26.2 mm to (119.0, 135.0)
- moved U10 1.41 mm to (119.0, 154.0)
- moved U2 1.41 mm to (81.0, 116.0)
- moved U1 1.28 mm to (90.5, 93.0)
- moved SW1 1.01 mm to (126.5, 100.8)
Routing:
- net S7: track 41.6 -> 87.6 mm, vias 1 -> 2
- net S8: track 61.8 -> 105.9 mm, vias 1 -> 2
- net DIN_5V: track 54.3 -> 29.1 mm
- net S4: track 40.6 -> 65.5 mm, vias 1 -> 2
- net Net-(U7-DOUT): track 57.2 -> 32.3 mm, vias 0 -> 2
- net Net-(U10-DIN): track 25.0 -> 48.4 mm, vias 0 -> 2
- net S5: track 55.6 -> 75.1 mm, vias 1 -> 2
- net S1: track 26.7 -> 40.5 mm
- net Net-(U8-DOUT): track 27.4 -> 16.7 mm, vias 0 -> 2
- net +5V: track 231.8 -> 223.8 mm
- net Net-(U3-DOUT): track 25.0 -> 30.4 mm, vias 0 -> 2
- net Net-(U4-DOUT): track 57.2 -> 52.4 mm, vias 0 -> 4
- net Net-(U6-DOUT): track 24.8 -> 29.2 mm, vias 0 -> 2
- net S9: track 82.3 -> 86.4 mm, vias 1 -> 2
- net S2: track 49.2 -> 45.7 mm, vias 1 -> 2
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Other:
- board size 56 x 83 mm -> 56 x 83.3 mm
- board text added: "JLCJLCJLC"
