File: Mini_Tastatur.kicad_sch (KiCad schematic)
At the start: 16 parts, among them IC1 74HCT1G125GW,125, SW1 RotaryEncoder_Switch, SW2 SW_Reset, U1 DM-OLED096-636, U10 MX1A-11NN_RGB, U2 MX1A-11NN_RGB, U3 MX1A-11NN_RGB, U4 MX1A-11NN_RGB, U5 MX1A-11NN_RGB, U6 MX1A-11NN_RGB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

Commit message: v2
Parts:
- D10: footprint Diode_SMD:D_MiniMELF -> Diode_SMD:D_SOD-523
- IC1: footprint Package_TO_SOT_SMD:SOT-353_SC-70-5 -> SOT65P212X110-5N
- U1: footprint SSD1306:MODULE_DM-OLED096-636 -> DM-OLED096-636:MODULE_DM-OLED096-636
Changed lines of the file:
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@@
 			)
 		)
-		(property "Footprint" "Diode_SMD:D_MiniMELF"
+		(property "Footprint" "Diode_SMD:D_SOD-523"
 			(at 146.05 131.445 0)
 			(effects
@@
 			)
 		)
-		(property "Description" "75V 0.15A Fast switching Diode, SOD-80"
+		(property "Description" "75V 0.15A Fast switching Diode, SOD-523"
 			(at 146.05 135.89 0)
 			(effects
@@
 			)
 		)
-		(property "Footprint" "Package_TO_SOT_SMD:SOT-353_SC-70-5"
+		(property "Footprint" "SOT65P212X110-5N"
 			(at 153.67 172.39 0)
 			(effects
@@
 			)
 		)
-		(property "Footprint" "SSD1306:MODULE_DM-OLED096-636"
+		(property "Footprint" "DM-OLED096-636:MODULE_DM-OLED096-636"
 			(at 144.78 53.34 0)
 			(effects
